Commit message: Fix trolley

File: urdf/trolley.xacro.urdf (robot description, URDF)
Before this commit: robot omnidirectional_robot, 4 links, 3 joints
Joints:
- joint wheel_2_joint: origin xyz=-0.106 0.106 0 rpy=1.57 0.0 0.785398 -> xyz=-0.075 0.12990381056 0 rpy=1.57 0.0 0.5235987755983
- joint wheel_3_joint: origin xyz=-0.106 -0.106 0 rpy=1.57 0.0 -0.785398 -> xyz=-0.075 -0.12990381056 0 rpy=1.57 0.0 -0.5235987755983

Commit message: Fixed omuni position and direction

File: urdf/trolley.xacro.urdf (robot description, URDF)
Before this commit: robot omnidirectional_robot, 4 links, 3 joints
Joints:
- joint wheel_1_joint: origin xyz=0.15 0 0.0 rpy=1.57 0.0 1.57 -> xyz=0.075 0.12990381056 0 rpy=1.57 0.0 -0.5235987755983
- joint wheel_2_joint: origin xyz=-0.075 0.12990381056 0 rpy=1.57 0.0 0.5235987755983 -> xyz=-0.15 0 0.0 rpy=1.57 0.0 1.57
- joint wheel_3_joint: origin xyz=-0.075 -0.12990381056 0 rpy=1.57 0.0 -0.5235987755983 -> xyz=0.075 -0.12990381056 0 rpy=1.57 0.0 -2.6179938779915

Commit message: Fixed wheel radius to 0.03m

File: urdf/trolley.xacro.urdf (robot description, URDF)
Before this commit: robot omnidirectional_robot, 4 links, 3 joints
Links:
- link wheel_1: geometry collision cylinder length=0.02 radius=0.05; visual cylinder length=0.02 radius=0.03
- link wheel_2: geometry collision cylinder length=0.02 radius=0.05; visual cylinder length=0.02 radius=0.03
- link wheel_3: geometry collision cylinder length=0.02 radius=0.05; visual cylinder length=0.02 radius=0.03

Commit message: Added lidar settings to urdf file

File: urdf/trolley.xacro.urdf (robot description, URDF)
Before this commit: robot omnidirectional_robot, 4 links, 3 joints
Links:
- added link lidar_link, mass 0.5; visual cylinder length=0.05 radius=0.05
Joints:
- added joint lidar_joint: type fixed, parent base_link, child lidar_link, origin xyz=0.15 0 0 rpy=0 0 0
- joint wheel_3_joint: axis 0.0 0.0 1.0 -> (none)

Commit message: Added robot on field

File: urdf/trolley.xacro.urdf (robot description, URDF)
Before this commit: robot omnidirectional_robot, 5 links, 4 joints
Links:
- link wheel_1: geometry collision cylinder length=0.02 radius=0.03; visual cylinder length=0.02 radius=0.03
- link wheel_2: geometry collision cylinder length=0.02 radius=0.03; visual cylinder length=0.02 radius=0.03
- link wheel_3: geometry collision cylinder length=0.02 radius=0.03; visual cylinder length=0.02 radius=0.03

Commit message: Added base_footprint

File: urdf/trolley.xacro.urdf (robot description, URDF)
Before this commit: robot omnidirectional_robot, 5 links, 4 joints
Links:
- added link base_footprint
Joints:
- added joint base_joint: type fixed, parent base_link, child base_footprint, origin xyz=0.0 0.0 -0.03 rpy=0 0 0

Commit message: Fixed invert

File: urdf/trolley.xacro.urdf (robot description, URDF)
Before this commit: robot omnidirectional_robot, 6 links, 5 joints
Links:
- removed link lidar_link
- added link base_laser, mass 0.5; visual cylinder length=0.05 radius=0.05
Joints:
- joint base_joint: child base_footprint -> base_link; origin xyz=0.0 0.0 -0.03 rpy=0 0 0 -> xyz=0.0 0.0 0.03 rpy=0 0 0; parent base_link -> base_footprint
- joint lidar_joint: child lidar_link -> base_laser
- joint wheel_3_joint: axis (none) -> 0.0 0.0 1.0
