Commit message: Fixed urdf file and Added drive program

File: urdf/diff.xacro.urdf (robot description, URDF)
Before this commit: robot diff_drive, 6 links, 5 joints
Links:
- link left_wheel: mass 0.1 -> 1
- link right_wheel: mass 0.1 -> 1
Joints:
- joint left_wheel_joint: origin xyz=0.04 0.06 0.0 rpy=1.57 0.0 0.0 -> xyz=0.03 0.06 0.0 rpy=1.57 0.0 0.0
- joint right_wheel_joint: origin xyz=0.04 -0.06 0.0 rpy=1.57 0.0 0.0 -> xyz=0.03 -0.06 0.0 rpy=1.57 0.0 0.0

Commit message: Added Lidar to diff robot

File: urdf/diff.xacro.urdf (robot description, URDF)
Before this commit: robot diff_drive, 6 links, 5 joints
Joints:
- joint lidar_joint: origin xyz=-0.075 0.0 0.0 rpy=0.0 0.0 0.157 -> xyz=-0.080 0.0 0.0 rpy=0.0 0.0 0.0
