Commit message: Fixed pertical filter bug

File: urdf/robot.xacro (robot description, xacro)
@@ -1,58 +1,90 @@
 <?xml version="1.0"?>
 <robot name="robot" xmlns:xacro="http://www.ros.org/wiki/xacro">
+  <!-- インクルード -->
   <xacro:include filename="$(find inrof2025_ros)/urdf/materials.xacro" />
   <xacro:include filename="$(find inrof2025_ros)/urdf/robot.trans" />
-  <link name="base_footprint"/>
+  <!-- base_footprint（地面接触用、摩擦のみ設定） -->
+  <link name="base_footprint">
+    <gazebo>
+      <surface>
+        <friction>
+          <ode>
+            <mu>1.0</mu>
+            <mu2>1.0</mu2>
+          </ode>
+        </friction>
+      </surface>
+    </gazebo>
+  </link>
+  <!-- base_link -->
   <link name="base_link">
     <inertial>
-      <origin xyz="-9.089504425782191e-15 -4.445651237390906e-17 4.545678390232227e-15" rpy="0 0 0" />
-      <mass value="0.012946126118149015" />
-      <inertia ixx="2.1e-05" iyy="0.0" izz="2.1e-05" ixy="-0.0" iyz="0.0" ixz="0.0" />
-    </inertial>
-    <visual>
-      <origin xyz="0 0 0" rpy="0 0 0" />
-      <geometry>
-        <mesh filename="file://$(find inrof2025_ros)/meshes/base_link.stl" scale="0.001 0.001 0.001" />
-      </geometry>
-      <material name="aluminum_satin" />
-    </visual>
-    <collision>
-      <origin xyz="0 0 0" rpy="0 0 0" />
-      <geometry>
-        <mesh filename="file://$(find inrof2025_ros)/meshes/base_link.stl" scale="0.001 0.001 0.001" />
-      </geometry>
-    </collision>
+      <origin xyz="-9.089504425782191e-15 -4.445651237390906e-17 4.545678390232227e-15" rpy="0 0 0"/>
+      <mass value="0.012946126118149015"/>
+      <!-- iyy をゼロから ixx と同じスケールに修正 -->
+      <inertia
+        ixx="2.1e-05"
+        iyy="2.1e-05"
+        izz="2.1e-05"
+        ixy="0.0"
+        iyz="0.0"
+        ixz="0.0"/>
+    </inertial>
+    <visual>
+      <origin xyz="0 0 0" rpy="0 0 0"/>
+      <geometry>
+        <mesh filename="file://$(find inrof2025_ros)/meshes/base_link.stl" scale="0.001 0.001 0.001"/>
+      </geometry>
+      <material name="aluminum_satin"/>
+    </visual>
+    <collision name="base_link_collision">
+      <origin xyz="0 0 0" rpy="0 0 0"/>
+      <geometry>
+        <mesh filename="file://$(find inrof2025_ros)/meshes/base_link.stl" scale="0.001 0.001 0.001"/>
+      </geometry>
+    </collision>
+    <gazebo reference="base_link_collision">
+      <surface>
+        <friction>
+          <ode>
+            <mu>1.0</mu>
+            <mu2>1.0</mu2>
+          </ode>
+        </friction>
+      </surface>
+    </gazebo>
   </link>
   <joint name="base_joint" type="fixed">
     <parent link="base_footprint"/>
-    <child link="base_link"/>
+    <child  link="base_link"/>
     <origin xyz="0.0 0.0 0.03" rpy="0 0 0"/>
   </joint>
+  <!-- LD19_with_mounter_v4_1 -->
   <link name="LD19_with_mounter_v4_1">
     <inertial>
-      <origin xyz="0.025278982742592118 0.01287150469895035 -0.022981220041423615" rpy="0 0 0" />
-      <mass value="0.19341283989224745" />
-      <inertia ixx="6.5e-05" iyy="7.9e-05" izz="8.9e-05" ixy="0.0" iyz="0.0" ixz="1.2e-05" />
-    </inertial>
-    <visual>
-      <origin xyz="-0.005 0.013 -0.0" rpy="0 0 0" />
-      <geometry>
-        <mesh filename="file://$(find inrof2025_ros)/meshes/LD19_with_mounter_v4_1.stl"
-          scale="0.001 0.001 0.001" />
-      </geometry>
-      <material name="steel_satin" />
-    </visual>
-    <!-- <collision>
-      <origin xyz="-0.005 0.013 -0.0" rpy="0 0 0" />
-      <geometry>
-        <mesh filename="file://$(find inrof2025_ros)/meshes/LD19_with_mounter_v4_1.stl"
-          scale="0.001 0.001 0.001" />
-      </geometry>
-    </collision> -->
-  </link>
+      <origin xyz="0.025278982742592118 0.01287150469895035 -0.022981220041423615" rpy="0 0 0"/>
+      <mass value="0.19341283989224745"/>
+      <inertia
+        ixx="6.5e-05"
+        iyy="7.9e-05"
+        izz="8.9e-05"
+        ixy="0.0"
+        iyz="0.0"
+        ixz="1.2e-05"/>
+    </inertial>
+    <visual>
+      <origin xyz="-0.005 0.013 -0.0" rpy="0 0 0"/>
+      <geometry>
+        <mesh filename="file://$(find inrof2025_ros)/meshes/LD19_with_mounter_v4_1.stl" scale="0.001 0.001 0.001"/>
+      </geometry>
+      <material name="steel_satin"/>
+    </visual>
+    <!-- collision が不要ならコメントアウトのままでOK -->
+  </link>
+  <!-- LiDAR -->
   <link name="lidar_link"/>
   <joint name="lidar_joint" type="fixed">
     <parent link="LD19_with_mounter_v4_1"/>
-    <child link="lidar_link"/>
+    <child  link="lidar_link"/>
     <origin xyz="0.03 0.013 -0.05" rpy="0 0 0"/>
   </joint>
@@ -66,7 +98,7 @@
           <horizontal>
             <samples>360</samples>
-            <resolution>1.000000</resolution>
+            <resolution>1.0</resolution>
             <min_angle>-1.570000</min_angle>
-            <max_angle>1.570000</max_angle>
+            <max_angle> 1.570000</max_angle>
           </horizontal>
         </scan>
@@ -91,146 +123,221 @@
     </sensor>
   </gazebo>
+  <!-- chassis_unit_v12_1 -->
   <link name="chassis_unit_v12_1">
     <inertial>
-      <origin xyz="-0.03167569261038175 -0.020149624242172634 -0.026142686915341103" rpy="0 0 0" />
-      <mass value="0.9094540640488471" />
-      <inertia ixx="0.000711" iyy="0.000485" izz="0.000788" ixy="0.000195" iyz="5.2e-05"
-        ixz="-3e-05" />
-    </inertial>
-    <visual>
-      <origin xyz="-0.0 0.045 0.005" rpy="0 0 0" />
-      <geometry>
-        <mesh filename="file://$(find inrof2025_ros)/meshes/chassis_unit_v12_1.stl"
-          scale="0.001 0.001 0.001" />
-      </geometry>
-      <material name="silicone_white" />
-    </visual>
-    <collision>
-      <origin xyz="-0.0 0.045 0.005" rpy="0 0 0" />
-      <geometry>
-        <mesh filename="file://$(find inrof2025_ros)/meshes/chassis_unit_v12_1.stl"
-          scale="0.001 0.001 0.001" />
-      </geometry>
-    </collision>
-  </link>
+      <origin xyz="-0.03167569261038175 -0.020149624242172634 -0.026142686915341103" rpy="0 0 0"/>
+      <mass value="0.9094540640488471"/>
+      <inertia
+        ixx="0.000711"
+        iyy="0.000485"
+        izz="0.000788"
+        ixy="0.000195"
+        iyz="0.000052"
+        ixz="0.000030"/>
+    </inertial>
+    <visual>
+      <origin xyz="-0.0 0.045 0.005" rpy="0 0 0"/>
+      <geometry>
+        <mesh filename="file://$(find inrof2025_ros)/meshes/chassis_unit_v12_1.stl" scale="0.001 0.001 0.001"/>
+      </geometry>
+      <material name="silicone_white"/>
+    </visual>
+    <collision name="chassis_unit_v12_1_collision">
+      <origin xyz="-0.0 0.045 0.005" rpy="0 0 0"/>
+      <geometry>
+        <mesh filename="file://$(find inrof2025_ros)/meshes/chassis_unit_v12_1.stl" scale="0.001 0.001 0.001"/>
+      </geometry>
+    </collision>
+    <gazebo reference="chassis_unit_v12_1_collision">
+      <surface>
+        <friction>
+          <ode>
+            <mu>1.0</mu>
+            <mu2>1.0</mu2>
+          </ode>
+        </friction>
+      </surface>
+    </gazebo>
+  </link>
+  <!-- chassis_unit_v12_2 -->
   <link name="chassis_unit_v12_2">
     <inertial>
-      <origin xyz="-0.03166397328252324 0.005142858085078819 -0.0261426869153411" rpy="0 0 0" />
-      <mass value="0.9094540640488471" />
-      <inertia ixx="0.000711" iyy="0.000486" izz="0.000788" ixy="-0.000195" iyz="-5.2e-05"
-        ixz="-3e-05" />
-    </inertial>
-    <visual>
-      <origin xyz="-0.0 -0.06 0.005" rpy="0 0 0" />
-      <geometry>
-        <mesh filename="file://$(find inrof2025_ros)/meshes/chassis_unit_v12_2.stl"
-          scale="0.001 0.001 0.001" />
-      </geometry>
-      <material name="silicone_white" />
-    </visual>
-    <collision>
-      <origin xyz="-0.0 -0.06 0.005" rpy="0 0 0" />
-      <geometry>
-        <mesh filename="file://$(find inrof2025_ros)/meshes/chassis_unit_v12_2.stl"
-          scale="0.001 0.001 0.001" />
-      </geometry>
-    </collision>
-  </link>
+      <origin xyz="-0.03166397328252324 0.005142858085078819 -0.0261426869153411" rpy="0 0 0"/>
+      <mass value="0.9094540640488471"/>
+      <inertia
+        ixx="0.000711"
+        iyy="0.000486"
+        izz="0.000788"
+        ixy="-0.000195"
+        iyz="-0.000052"
+        ixz="-0.000030"/>
+    </inertial>
+    <visual>
+      <origin xyz="-0.0 -0.06 0.005" rpy="0 0 0"/>
+      <geometry>
+        <mesh filename="file://$(find inrof2025_ros)/meshes/chassis_unit_v12_2.stl" scale="0.001 0.001 0.001"/>
+      </geometry>
+      <material name="silicone_white"/>
+    </visual>
+    <collision name="chassis_unit_v12_2_collision">
+      <origin xyz="-0.0 -0.06 0.005" rpy="0 0 0"/>
+      <geometry>
+        <mesh filename="file://$(find inrof2025_ros)/meshes/chassis_unit_v12_2.stl" scale="0.001 0.001 0.001"/>
+      </geometry>
+    </collision>
+    <gazebo reference="chassis_unit_v12_2_collision">
+      <surface>
+        <friction>
+          <ode>
+            <mu>1.0</mu>
+            <mu2>1.0</mu2>
+          </ode>
+        </friction>
+      </surface>
+    </gazebo>
+  </link>
+  <!-- alm_1_v3_1 -->
   <link name="alm_1_v3_1">
     <inertial>
-      <origin xyz="-0.051961049228441504 0.029999999552957693 0.004999999999999994" rpy="0 0 0" />
-      <mass value="0.01316675074543267" />
-      <inertia ixx="6e-06" iyy="1.6e-05" izz="2.1e-05" ixy="9e-06" iyz="0.0" ixz="-0.0" />
-    </inertial>
-    <visual>
-      <origin xyz="0.051962 0.09 0.005" rpy="0 0 0" />
-      <geometry>
-        <mesh filename="file://$(find inrof2025_ros)/meshes/alm_1_v3_1.stl"
-          scale="0.001 0.001 0.001" />
-      </geometry>
-      <material name="aluminum_satin" />
-    </visual>
-    <collision>
-      <origin xyz="0.051962 0.09 0.005" rpy="0 0 0" />
-      <geometry>
-        <mesh filename="file://$(find inrof2025_ros)/meshes/alm_1_v3_1.stl"
-          scale="0.001 0.001 0.001" />
-      </geometry>
-    </collision>
-  </link>
+      <origin xyz="-0.051961049228441504 0.029999999552957693 0.004999999999999994" rpy="0 0 0"/>
+      <mass value="0.01316675074543267"/>
+      <inertia
+        ixx="6e-06"
+        iyy="1.6e-05"
+        izz="2.1e-05"
+        ixy="9e-06"
+        iyz="0.0"
+        ixz="0.0"/>
+    </inertial>
+    <visual>
+      <origin xyz="0.051962 0.09 0.005" rpy="0 0 0"/>
+      <geometry>
+        <mesh filename="file://$(find inrof2025_ros)/meshes/alm_1_v3_1.stl" scale="0.001 0.001 0.001"/>
+      </geometry>
+      <material name="aluminum_satin"/>
+    </visual>
+    <collision name="alm_1_v3_1_collision">
+      <origin xyz="0.051962 0.09 0.005" rpy="0 0 0"/>
+      <geometry>
+        <mesh filename="file://$(find inrof2025_ros)/meshes/alm_1_v3_1.stl" scale="0.001 0.001 0.001"/>
+      </geometry>
+    </collision>
+    <gazebo reference="alm_1_v3_1_collision">
+      <surface>
+        <friction>
+          <ode>
+            <mu>1.0</mu>
+            <mu2>1.0</mu2>
+          </ode>
+        </friction>
+      </surface>
+    </gazebo>
+  </link>
+  <!-- chassis_unit_v12_3 -->
   <link name="chassis_unit_v12_3">
     <inertial>
-      <origin xyz="-0.0016124325639870207 -0.03749323384290623 -0.02614268691534118" rpy="0 0 0" />
-      <mass value="0.9094540640488471" />
-      <inertia ixx="0.000373" iyy="0.000824" izz="0.000788" ixy="0.0" iyz="0.0" ixz="6e-05" />
-    </inertial>
-    <visual>
-      <origin xyz="0.142894 -0.0375 0.005" rpy="0 0 0" />
-      <geometry>
-        <mesh filename="file://$(find inrof2025_ros)/meshes/chassis_unit_v12_3.stl"
-          scale="0.001 0.001 0.001" />
-      </geometry>
-      <material name="silicone_white" />
-    </visual>
-    <collision>
-      <origin xyz="0.142894 -0.0375 0.005" rpy="0 0 0" />
-      <geometry>
-        <mesh filename="file://$(find inrof2025_ros)/meshes/chassis_unit_v12_3.stl"
-          scale="0.001 0.001 0.001" />
-      </geometry>
-    </collision>
-  </link>
+      <origin xyz="-0.0016124325639870207 -0.03749323384290623 -0.02614268691534118" rpy="0 0 0"/>
+      <mass value="0.9094540640488471"/>
+      <inertia
+        ixx="0.000373"
+        iyy="0.000824"
+        izz="0.000788"
+        ixy="0.0"
+        iyz="0.0"
+        ixz="6e-05"/>
+    </inertial>
+    <visual>
+      <origin xyz="0.142894 -0.0375 0.005" rpy="0 0 0"/>
+      <geometry>
+        <mesh filename="file://$(find inrof2025_ros)/meshes/chassis_unit_v12_3.stl" scale="0.001 0.001 0.001"/>
+      </geometry>
+      <material name="silicone_white"/>
+    </visual>
+    <collision name="chassis_unit_v12_3_collision">
+      <origin xyz="0.142894 -0.0375 0.005" rpy="0 0 0"/>
+      <geometry>
+        <mesh filename="file://$(find inrof2025_ros)/meshes/chassis_unit_v12_3.stl" scale="0.001 0.001 0.001"/>
+      </geometry>
+    </collision>
+    <gazebo reference="chassis_unit_v12_3_collision">
+      <surface>
+        <friction>
+          <ode>
+            <mu>1.0</mu>
+            <mu2>1.0</mu2>
+          </ode>
+        </friction>
+      </surface>
+    </gazebo>
+  </link>
+  <!-- alm_1_v3_2 -->
   <link name="alm_1_v3_2">
     <inertial>
-      <origin xyz="-0.051961049228450455 -0.02999999955294213 0.004999999999999977" rpy="0 0 0" />
-      <mass value="0.01316675074543267" />
-      <inertia ixx="6e-06" iyy="1.6e-05" izz="2.1e-05" ixy="-9e-06" iyz="0.0" ixz="0.0" />
-    </inertial>
-    <visual>
-      <origin xyz="0.051962 -0.09 0.005" rpy="0 0 0" />
-      <geometry>
-        <mesh filename="file://$(find inrof2025_ros)/meshes/alm_1_v3_2.stl"
-          scale="0.001 0.001 0.001" />
-      </geometry>
-      <material name="aluminum_satin" />
-    </visual>
-    <collision>
-      <origin xyz="0.051962 -0.09 0.005" rpy="0 0 0" />
-      <geometry>
-        <mesh filename="file://$(find inrof2025_ros)/meshes/alm_1_v3_2.stl"
-          scale="0.001 0.001 0.001" />
-      </geometry>
-    </collision>
-  </link>
+      <origin xyz="-0.051961049228450455 -0.02999999955294213 0.004999999999999977" rpy="0 0 0"/>
+      <mass value="0.01316675074543267"/>
+      <inertia
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
Commit message: Added simple slam

File: urdf/robot.xacro (robot description, xacro)
@@ -87,5 +87,5 @@
     <parent link="LD19_with_mounter_v4_1"/>
     <child  link="lidar_link"/>
-    <origin xyz="0.03 0.013 -0.05" rpy="0 0 0"/>
+    <origin xyz="0.0 0.013 -0.05" rpy="0 0 0"/>
   </joint>
   <gazebo reference="lidar_link">
@@ -99,6 +99,6 @@
             <samples>360</samples>
             <resolution>1.0</resolution>
-            <min_angle>-1.570000</min_angle>
-            <max_angle> 1.570000</max_angle>
+            <min_angle>-1.3</min_angle>
+            <max_angle> 1.3</max_angle>
           </horizontal>
         </scan>
@@ -111,5 +111,5 @@
           <type>gaussian</type>
           <mean>0.0</mean>
-          <stddev>0.01</stddev>
+          <stddev>0.0</stddev>
         </noise>
       </ray>
@@ -119,5 +119,5 @@
         </ros>
         <output_type>sensor_msgs/LaserScan</output_type>
-        <frameName>lidar_link</frameName>
+        <frame_name>lidar_link</frame_name>
       </plugin>
     </sensor>

Commit message: Fixed lidar reletive position

File: urdf/robot.xacro (robot description, xacro)
@@ -87,5 +87,5 @@
     <parent link="LD19_with_mounter_v4_1"/>
     <child  link="lidar_link"/>
-    <origin xyz="0.0 0.013 -0.05" rpy="0 0 0"/>
+    <origin xyz="0.033 0.013 -0.05" rpy="0 0 0"/>
   </joint>
   <gazebo reference="lidar_link">

Commit message: Added ldlidar node

File: urdf/robot.xacro (robot description, xacro)
@@ -83,5 +83,5 @@
   </link>
   <!-- LiDAR -->
-  <link name="lidar_link"/>
+  <link name="ldlidar_base"/>
   <joint name="lidar_joint" type="fixed">
     <parent link="LD19_with_mounter_v4_1"/>
@@ -89,5 +89,5 @@
     <origin xyz="0.033 0.013 -0.05" rpy="0 0 0"/>
   </joint>
-  <gazebo reference="lidar_link">
+  <gazebo reference="ldlidar_base">
     <sensor type="ray" name="lidar_sensor">
       <always_on>true</always_on>
@@ -116,8 +116,8 @@
       <plugin filename="libgazebo_ros_ray_sensor.so" name="gazebo_lidar">
         <ros>
-          <remapping>~/out:=scan</remapping>
+          <remapping>~/out:=/ldlidar_node/scan</remapping>
         </ros>
         <output_type>sensor_msgs/LaserScan</output_type>
-        <frame_name>lidar_link</frame_name>
+        <frame_name>ldlidar_base</frame_name>
       </plugin>
     </sensor>

Commit message: Fixed urdf file

File: urdf/robot.xacro (robot description, xacro)
@@ -86,5 +86,5 @@
   <joint name="lidar_joint" type="fixed">
     <parent link="LD19_with_mounter_v4_1"/>
-    <child  link="lidar_link"/>
+    <child  link="ldlidar_base"/>
     <origin xyz="0.033 0.013 -0.05" rpy="0 0 0"/>
   </joint>
